File: RPi_Zero_pHat_Template.sch (KiCad schematic (older format))
At the start: 2 parts, among them J1 RPi_GPIO, J2 RPi_GPIO

Commit message: Major update to KiCad 5.
Include symbol, footprints, and 3D models.
Parts:
- J1, J2: symbol RPi_Zero_pHat_Template-rescue:RPi_GPIO -> Connector-ML:RPi_GPIO
Other:
- note added: "Socket on bottom"
Changed lines of the file:
@@
 $EndDescr
 $Comp
-L RPi_Zero_pHat_Template-rescue:RPi_GPIO J1
+L Connector-ML:RPi_GPIO J1
 U 1 1 5515D39E
 P 2750 2700
@@
 $EndComp
 $Comp
-L RPi_Zero_pHat_Template-rescue:RPi_GPIO J2
+L Connector-ML:RPi_GPIO J2
 U 1 1 5516AE26
 P 7500 2700
@@
 	1    0    0    -1
 $EndComp
-Text Notes 2950 5000 0    60   Italic 0
+Text Notes 2550 5000 0    100  Italic 0
 Surface Mount Connector
-Text Notes 7800 5000 0    60   Italic 0
+Text Notes 7450 5000 0    100  Italic 0
 Thru-Hole Connector
+Text Notes 2550 5200 0    100  Italic 0
+Socket on bottom
 $EndSCHEMATC
